File: M68000.kicad_pcb (KiCad board)
At the start: 2 copper layers, 148 x 70.8 mm, 70 parts, among them J1 JTAG1, J2 USB_B, J3 DB9_Female_MountingHoles, J4 2nd DUART CHNL, SW1 Util_SW, SW2 RESET_SW, SW3 STEP_SW, U1 MAX699, U2 XC9572, U3 MC68000FN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

Commit message: Submitted to JLCPCB
Parts:
- added G***: LOGO, LOGO, F.Cu at (193.2, 84.6)
- added REF**: MountingHole_2.2mm_M2_DIN965_Pad, MountingHole:MountingHole_2.2mm_M2_DIN965_Pad, F.Cu at (200.1, 142.6)
- added REF**: MountingHole_2.2mm_M2_DIN965_Pad, MountingHole:MountingHole_2.2mm_M2_DIN965_Pad, F.Cu at (200.1, 77.2)
- added REF**: MountingHole_2.2mm_M2_DIN965_Pad, MountingHole:MountingHole_2.2mm_M2_DIN965_Pad, F.Cu at (57.4, 77.2)
- added REF**: MountingHole_2.2mm_M2_DIN965_Pad, MountingHole:MountingHole_2.2mm_M2_DIN965_Pad, F.Cu at (57.4, 142.6)
- R1, R2, R3, R5: value 330 -> 4.7k
- moved J2 1.50 mm to (57.1, 135.2)
- moved J1 0.25 mm to (198.0, 138.3)
- moved R18 0.07 mm to (179.2, 85.2), turned to 90 degrees
- moved R19 0.07 mm to (170.2, 85.2), turned to 90 degrees
Routing:
- net +5V: track 731.9 -> 724.6 mm
- net /R/~{W}: track 217.3 -> 216.1 mm
- net /ROM1_~{CS}: track 96.7 -> 95.7 mm
- net /USB_POWER: track 12.1 -> 12.8 mm
- net /SW_UTIL: track 31.1 -> 30.7 mm, vias 2 -> 0
Other:
- outline, holes or cut-outs redrawn
- board text added: "JLCJLCJLCJLC"
- board text added: "Jackson Miller MCD 2022"
- board text added: "M68000 Single Board Computer"
- board text added: "Made with"
- board text added: "github.com/jack-mil/m68000-pcb"
